Commit message: Update models

File: porthos_description/robots/porthos_description.xacro (robot description, xacro)
@@ -1,8 +1,8 @@
 <?xml version="1.0"?>
 <robot xmlns:xacro="http://ros.org/wiki/xacro" name="porthos_description">
-<xacro:include filename="$(find p2os_urdf)/defs/pioneer3at_body.xacro"/>
-<xacro:include filename="$(find cyton_description)/robots/cyton_gazebo_description.urdf"/>
-<xacro:include filename="$(find porthos_description)/robots/suporte_porthos_description.URDF"/>
-<xacro:include filename="$(find pr2_description)/urdf/sensors/kinect_camera.urdf.xacro" />
+<xacro:include filename="$(find porthos_description)/robots/pioneer3at_body.xacro"/>
+<!-- <xacro:include filename="$(find cyton_description)/robots/cyton_gazebo_description.urdf"/> -->
+<xacro:include filename="$(find porthos_description)/robots/suporte_porthos_description.urdf"/>
+<!-- <xacro:include filename="$(find pr2_description)/urdf/sensors/kinect_camera.urdf.xacro" /> -->
 <xacro:include filename="$(find pr2_description)/urdf/common.xacro" />
 <xacro:p3at_front suffix="left" reflect="1"/>
@@ -10,9 +10,9 @@
 <xacro:p3at_back suffix="left" reflect="1"/>
 <xacro:p3at_back suffix="right" reflect="-1"/>
-<joint name="pioneer2cyton" type="fixed">
+<!-- <joint name="pioneer2cyton" type="fixed">
 	<origin xyz="0.08 0.071 0.004" rpy="0 0 0"/>
 		<parent link="top_plate"/>
 		<child link="link0"/>
-</joint>
+</joint> -->
 <joint name="pioneer2suporte" type="fixed">
 	<origin xyz="0.073 0.160 0.004" rpy="0 0 -1.57"/>

File: porthos_description/robots/suporte_porthos_description.urdf (robot description, URDF)
Before this commit: robot suporte_porthos_description, 11 links, 10 joints
Links:
- removed link suporte_depth
- removed link tv
- link arm_control_box: mass 1.88580869219064 -> 0.45; geometry collision mesh filename=package://athos_description/meshes/arm_control_box_mesh.dae; visual mesh filename=package://athos_description/meshes/arm_control_box_mesh.dae
- link suporte_armControl: geometry collision mesh filename=package://athos_description/meshes/suporte_armControl_mesh.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; visual mesh filename=package://athos_description/meshes/suporte_armControl_mesh.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
- link suporte_base: mass 5 -> 0.5; geometry collision mesh filename=package://athos_description/meshes/suporte_base_mesh.dae; visual mesh filename=package://athos_description/meshes/suporte_base_mesh.dae
- link suporte_kinect: geometry collision mesh filename=package://athos_description/meshes/suporte_kinect_mesh.dae; visual mesh filename=package://athos_description/meshes/suporte_kinect_mesh.dae
- link suporte_monitor: geometry collision mesh filename=package://athos_description/meshes/suporte_monitor_mesh.dae; visual mesh filename=package://athos_description/meshes/suporte_monitor_mesh.dae
- link tampa1: geometry collision mesh filename=package://athos_description/meshes/tampa1_mesh.dae; visual mesh filename=package://athos_description/meshes/tampa1_mesh.dae
- link tampa2: geometry collision mesh filename=package://athos_description/meshes/tampa2_mesh.dae; visual mesh filename=package://athos_description/meshes/tampa2_mesh.dae
- link tampa3: geometry collision mesh filename=package://athos_description/meshes/tampa3_mesh.dae; visual mesh filename=package://athos_description/meshes/tampa3_mesh.dae
- link tampa4: geometry collision mesh filename=package://athos_description/meshes/tampa4_mesh.dae; visual mesh filename=package://athos_description/meshes/tampa4_mesh.dae
Joints:
- removed joint depth_joint
- removed joint suporte2tv
- joint armControl: origin xyz=0.03 -0.043 0.145 rpy=1.5708 0 0 -> xyz=0.161 -0.0743 0.1569 rpy=1.5708 0 0
- joint kinect_joint: origin xyz=0 -0.0429999999999997 0.6 rpy=1.5707963267949 0 0 -> xyz=0.161 -0.074 0.615 rpy=1.5707963267949 0 0
- joint monitor_joint: origin xyz=0.32 -0.103 0.335 rpy=-1.5707963267949 -6.12303176911189E-17 -1.5707963267949 -> xyz=0.16 -0.113 0.335 rpy=-1.5707963267949 3.14159265358979 -1.5707963267949
- joint suporte2controlbox: origin xyz=0.0728041142425171 -0.0429999999999999 0.175 rpy=1.5707963267949 0 0 -> xyz=0.16 -0.125 0.16 rpy=1.5707963267949 0 0
